File: Modulo 7/PCB/PCB.kicad_pcb (KiCad board)
At the start: 2 copper layers, 40.6 x 88.6 mm, 11 parts, among them J1 Batt, SW1 PowerBatt, SW2 WiFi, SW3 IP, U1 ESP32-DEVKIT-V1, U2 MAX30102

Commit message: Add files via upload
Parts:
- J1: footprint Connector_Wire:SolderWire-0.5sqmm_1x02_P4.6mm_D0.9mm_OD2.1mm -> Connector_JST:JST_XH_B2B-XH-A_1x02_P2.50mm_Vertical
- moved J1 10.1 mm to (132.1, 140.0)
Connections:
- U2 pad 1: unconnected-(U2-NC-Pad1) -> /GND
Routing:
- net /GND: track 135.1 -> 166.5 mm, vias 0 -> 2
- net /+: track 38.4 -> 36.3 mm
- net Net-(Brd1-SCL): track 67.2 -> 66.6 mm
- added copper zone on F.Cu, net (none)
Other:
- board size 40.6 x 88.6 mm -> 44 x 88.2 mm

Commit message: Add files via upload
Parts:
- R1, R2: footprint Resistor_SMD:R_0201_0603Metric -> Resistor_SMD:R_0805_2012Metric
- moved R2 2.08 mm to (132.4, 90.7)
- moved R1 0.99 mm to (132.6, 63.1)
Connections:
- U2 pad 4: /Vdd -> unconnected-(U2-PGND-Pad4)
Routing:
- net /GND: track 166.5 -> 164.1 mm, vias 2 -> 1
- net Net-(U1-D35): track 32.8 -> 34.4 mm
- net Net-(SW2-C): track 2.65 -> 4.06 mm
- net Net-(U1-VIN): track 79.2 -> 80.5 mm
