File: Modulo 7/PCB/PCB.kicad_sch (KiCad schematic)
At the start: 9 parts, among them J1 Batt, SW1 PowerBatt, SW2 WiFi, SW3 IP, U1 ESP32-DEVKIT-V1, U2 MAX30102

Commit message: Add files via upload
Parts:
- J1: footprint Connector_Wire:SolderWire-0.5sqmm_1x02_P4.6mm_D0.9mm_OD2.1mm -> Connector_JST:JST_XH_B2B-XH-A_1x02_P2.50mm_Vertical

Commit message: Add files via upload
Parts:
- R1, R2: footprint Resistor_SMD:R_0201_0603Metric -> Resistor_SMD:R_0805_2012Metric
Changed lines of the file:
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@@
       (effects (font (size 1.27 1.27)))
     )
-    (property "Footprint" "Resistor_SMD:R_0201_0603Metric" (at 146.05 42.418 90)
+    (property "Footprint" "Resistor_SMD:R_0805_2012Metric" (at 146.05 42.418 90)
       (effects (font (size 1.27 1.27)) hide)
     )
@@
       (effects (font (size 1.27 1.27)) (justify right))
     )
-    (property "Footprint" "Resistor_SMD:R_0201_0603Metric" (at 249.428 90.17 90)
+    (property "Footprint" "Resistor_SMD:R_0805_2012Metric" (at 249.428 90.17 90)
       (effects (font (size 1.27 1.27)) hide)
     )
